Commit message: add camera urdf

File: src/my_robot/urdf/my_robot.xacro (robot description, xacro)
@@ -29,4 +29,7 @@
         <box size=".4 .2 .1"/>
       </geometry>
+      <material name = ''>
+        <color rgba="0.75294 0.75294 0.75294 1"/>
+      </material>
     </visual>
     <collision name='back_caster_collision'>
@@ -117,3 +120,32 @@
     <dynamics damping="1.0" friction="1.0"/>
   </joint>
+  <link name='camera'>
+    <inertial>
+      <mass value="0.10"/>
+      <origin xyz="0.0 0 0" rpy=" 0 0 0"/>
+      <inertia
+          ixx="1e-6" ixy="0" ixz="0"
+          iyy="1e-6" iyz="0"
+          izz="1e-6"
+      />
+    </inertial>
+    <collision>
+      <origin xyz="0 0 0" rpy=" 0 0 0"/>
+      <geometry>
+        <box size=".05 .05 .05"/>
+      </geometry>
+    </collision>
+    <visual>
+      <origin xyz="0 0 0" rpy=" 0 0 0"/>
+      <geometry>
+        <box size=".05 .05 .05"/>
+      </geometry>
+    </visual>
+  </link>
+  <joint type="fixed" name="camera_joint">
+    <origin xyz="0.2 0 0" rpy="0 0 0"/>
+    <child link="camera"/>
+    <parent link="chassis"/>
+    <axis xyz="0 1 0" rpy="0 0 0"/>
+  </joint>
 </robot>

Commit message: add laser scan urdf

File: src/my_robot/urdf/my_robot.xacro (robot description, xacro)
@@ -79,4 +79,7 @@
         <cylinder length="0.05" radius="0.1"/>
       </geometry>
+      <material name="Cyan">
+        <color rgba = "0 1 1 1"/>
+      </material>
     </visual>
   </link>
@@ -110,4 +113,7 @@
         <cylinder length="0.05" radius="0.1"/>
       </geometry>
+      <material name="Cyan">
+        <color rgba = "0 1 1 1"/>
+      </material>
     </visual>
   </link>
@@ -149,3 +155,32 @@
     <axis xyz="0 1 0" rpy="0 0 0"/>
   </joint>
+  <link name='hokuyo'>
+    <inertial>
+      <mass value="1e-5"/>
+      <origin xyz="0.0 0 0" rpy=" 0 0 0"/>
+      <inertia
+          ixx="1e-6" ixy="0" ixz="0"
+          iyy="1e-6" iyz="0"
+          izz="1e-6"
+      />
+    </inertial>
+    <collision>
+      <origin xyz="0 0 0" rpy=" 0 0 0"/>
+      <geometry>
+        <box size=".1 .1 .1"/>
+      </geometry>
+    </collision>
+    <visual>
+      <origin xyz="0 0 0" rpy=" 0 0 0"/>
+      <geometry>
+        <mesh filename ="package://my_robot/meshes/hokuyo.dae" />
+      </geometry>
+    </visual>
+  </link>
+  <joint type="fixed" name="hokuyo_joint">
+    <origin xyz="0.15 0 0.1" rpy="0 0 0"/>
+    <child link="hokuyo"/>
+    <parent link="chassis"/>
+    <axis xyz="0 1 0" rpy="0 0 0"/>
+  </joint>
 </robot>
